Commit message: chore!: rename (#2)

File: j6_gen1_description/urdf/vehicle.xacro (robot description, xacro)
@@ -2,5 +2,5 @@
 <robot xmlns:xacro="http://ros.org/wiki/xacro">
   <!-- load parameter -->
-  <xacro:property name="vehicle_info" value="${xacro.load_yaml('$(find j6_description)/config/vehicle_info.param.yaml')}"/>
+  <xacro:property name="vehicle_info" value="${xacro.load_yaml('$(find j6_gen1_description)/config/vehicle_info.param.yaml')}"/>
   <!-- vehicle body -->
   <link name="base_link">
@@ -8,5 +8,5 @@
       <origin xyz="0 0 0" rpy="0.0 0.0 0.0"/>
       <geometry>
-        <mesh filename="package://j6_description/mesh/BYD_J6.dae" scale="1 1 1"/>
+        <mesh filename="package://j6_gen1_description/mesh/BYD_J6.dae" scale="1 1 1"/>
       </geometry>
     </visual>
